Commit message: Remove unused driver launch files

File: description/voxel.urdf.xacro (robot description, xacro)
@@ -18,8 +18,8 @@
       <visual>
         <geometry>
-          <box size="0.003 0.080 .020"/>
+          <box size="0.003 0.090 .020"/>
         </geometry>
         <material name="gray">
-          <color rgba="0.7 0.7 0.7 1"/>
+          <color rgba="0.1 0.1 0.1 1"/>
         </material>
       </visual>
@@ -28,7 +28,7 @@
       <visual>
         <geometry>
-          <cylinder length="0.020" radius="0.008"/>
+          <cylinder length="0.016" radius="0.008"/>
         </geometry>
-        <origin xyz="0.012 0 0" rpy="0 ${M_PI/2} 0"/>
+        <origin xyz="-0.008 0 0" rpy="0 ${M_PI/2} 0"/>
         <material name="black">
           <color rgba="0 0 0 1"/>
@@ -41,7 +41,7 @@
       <visual>
         <geometry>
-          <cylinder length="0.020" radius="0.008"/>
+          <cylinder length="0.016" radius="0.008"/>
         </geometry>
-        <origin xyz="0.012 0 0" rpy="0 ${M_PI/2} 0"/>
+        <origin xyz="-0.008 0 0" rpy="0 ${M_PI/2} 0"/>
         <material name="black">
           <color rgba="0 0 0 1"/>
@@ -96,5 +96,5 @@
       <parent link="${name}_camera"/>
       <child link="${name}_left_frame"/>
-      <origin xyz="0 ${INTEROCULAR/2} 0"/>
+      <origin xyz="0.016 ${INTEROCULAR/2} 0"/>
     </joint>
     <joint name="${name}_left_frame_to_${name}_left_optical_frame" type="fixed">
@@ -106,5 +106,5 @@
       <parent link="${name}_camera"/>
       <child link="${name}_right_frame"/>
-      <origin xyz="0 -${INTEROCULAR/2} 0"/>
+      <origin xyz="0.016 -${INTEROCULAR/2} 0"/>
     </joint>
     <joint name="${name}_right_frame_to_${name}_right_optical_frame" type="fixed">

Commit message: Add calibration files

File: description/voxel.urdf.xacro (robot description, xacro)
@@ -51,41 +51,4 @@
     <link name="${name}_right_optical_frame">
     </link>
-  <!--
-    <link name="base_laser">
-      <visual>
-        <geometry>
-          <cylinder length="0.02" radius="0.04"/>
-        </geometry>
-      </visual>
-    </link>
-    <link name="camera_link">
-      <visual>
-        <geometry>
-          <box size="0.06 .28 .03"/>
-        </geometry>
-        <origin rpy="0 0.05 0" xyz="-0.03 0 0"/>
-      </visual>
-    </link>
-    <link name="top_plate">
-      <visual>
-        <geometry>
-          <box size="0.326 0.206 .003"/>
-        </geometry>
-        <origin xyz="0 0 -0.0015"/>
-        <material name="polycarb">
-          <color rgba="1 1 1 0.4"/>
-        </material>
-      </visual>
-    </link>
-    <joint name="base_link_to_camera_link" type="fixed">
-      <parent link="base_link"/>
-      <child link="camera_link"/>
-      <origin rpy="0 -0.05 0" xyz="-0.112 0.0 0.230"/>
-    </joint>
-    <joint name="base_link_to_top_plate" type="fixed">
-      <parent link="base_link"/>
-      <child link="top_plate"/>
-      <origin xyz="0 0.0 0.147"/>
-    </joint> -->
     <joint name="${name}_to_${name}_camera" type="fixed">
       <parent link="${name}"/>
