Commit message: Update everything for the ELP dual lens camera

File: description/voxel_camera.urdf.xacro (robot description, xacro)
@@ -1,7 +1,9 @@
 <?xml version="1.0"?>
-<robot name="voxel" xmlns:xacro="http://ros.org/wiki/xacro">
+<robot name="voxel_camera" xmlns:xacro="http://ros.org/wiki/xacro">
   <xacro:property name="M_PI" value="3.1415926535897931" />
-  <xacro:property name="INTEROCULAR" value="0.065" />
-  <xacro:macro name="voxel" params="name">
+  <xacro:property name="INTEROCULAR" value="0.060" />
+  <xacro:property name="BOARD_THICKNESS" value="0.002" />
+  <xacro:property name="LENS_LENGTH" value="0.014" />
+  <xacro:macro name="voxel_camera" params="name">
     <link name="${name}">
       <visual>
@@ -15,8 +17,8 @@
       </visual>
     </link>
-    <link name="${name}_camera">
+    <link name="${name}_pcb">
       <visual>
         <geometry>
-          <box size="0.003 0.090 .020"/>
+          <box size="0.002 0.070 .016"/>
         </geometry>
         <material name="gray">
@@ -28,7 +30,7 @@
       <visual>
         <geometry>
-          <cylinder length="0.016" radius="0.008"/>
+          <cylinder length="${LENS_LENGTH}" radius="0.005"/>
         </geometry>
-        <origin xyz="-0.008 0 0" rpy="0 ${M_PI/2} 0"/>
+        <origin xyz="${-LENS_LENGTH/2} 0 0" rpy="0 ${M_PI/2} 0"/>
         <material name="black">
           <color rgba="0 0 0 1"/>
@@ -41,7 +43,7 @@
       <visual>
         <geometry>
-          <cylinder length="0.016" radius="0.008"/>
+          <cylinder length="${LENS_LENGTH}" radius="0.005"/>
         </geometry>
-        <origin xyz="-0.008 0 0" rpy="0 ${M_PI/2} 0"/>
+        <origin xyz="${-LENS_LENGTH/2} 0 0" rpy="0 ${M_PI/2} 0"/>
         <material name="black">
           <color rgba="0 0 0 1"/>
@@ -51,13 +53,13 @@
     <link name="${name}_right_optical_frame">
     </link>
-    <joint name="${name}_to_${name}_camera" type="fixed">
+    <joint name="${name}_to_${name}_pcb" type="fixed">
       <parent link="${name}"/>
-      <child link="${name}_camera"/>
+      <child link="${name}_pcb"/>
       <origin xyz="-0.010 0 0"/>
     </joint>
-    <joint name="${name}_camera_to_${name}_left_frame" type="fixed">
-      <parent link="${name}_camera"/>
+    <joint name="${name}_pcb_to_${name}_left_frame" type="fixed">
+      <parent link="${name}_pcb"/>
       <child link="${name}_left_frame"/>
-      <origin xyz="0.016 ${INTEROCULAR/2} 0"/>
+      <origin xyz="${BOARD_THICKNESS/2 + LENS_LENGTH} ${INTEROCULAR/2} 0"/>
     </joint>
     <joint name="${name}_left_frame_to_${name}_left_optical_frame" type="fixed">
@@ -66,8 +68,8 @@
       <origin xyz="0 0 0" rpy="${-M_PI/2} 0 ${-M_PI/2}"/>
     </joint>
-    <joint name="${name}_camera_to_${name}_right_frame" type="fixed">
-      <parent link="${name}_camera"/>
+    <joint name="${name}_pcb_to_${name}_right_frame" type="fixed">
+      <parent link="${name}_pcb"/>
       <child link="${name}_right_frame"/>
-      <origin xyz="0.016 -${INTEROCULAR/2} 0"/>
+      <origin xyz="${BOARD_THICKNESS/2 + LENS_LENGTH} ${-INTEROCULAR/2} 0"/>
     </joint>
     <joint name="${name}_right_frame_to_${name}_right_optical_frame" type="fixed">

File: description/voxel_standalone.urdf.xacro (robot description, xacro)
@@ -2,6 +2,6 @@
 <robot name="voxel_standalone" xmlns:xacro="http://ros.org/wiki/xacro">
   <!-- include the voxel macro -->
-  <xacro:include filename="$(find voxel)/description/voxel.urdf.xacro"/>
+  <xacro:include filename="$(find voxel)/description/voxel_camera.urdf.xacro"/>
   <!-- use the voxel macro to create a camera with name "voxel" -->
-  <voxel name="voxel"/>
+  <voxel_camera name="voxel"/>
 </robot>
