Commit message: Rename package from voxel to elp_stereo_camera

File: description/elp_stereo_camera.urdf.xacro (robot description, xacro)
@@ -1,9 +1,9 @@
 <?xml version="1.0"?>
-<robot name="voxel_camera" xmlns:xacro="http://ros.org/wiki/xacro">
+<robot name="elp_stereo_camera" xmlns:xacro="http://ros.org/wiki/xacro">
   <xacro:property name="M_PI" value="3.1415926535897931" />
   <xacro:property name="INTEROCULAR" value="0.060" />
   <xacro:property name="BOARD_THICKNESS" value="0.002" />
   <xacro:property name="LENS_LENGTH" value="0.014" />
-  <xacro:macro name="voxel_camera" params="name">
+  <xacro:macro name="elp_stereo_camera" params="name">
     <link name="${name}">
       <visual>

Commit message: Remove plastic enclosure from camera macro

File: description/elp_stereo_camera.urdf.xacro (robot description, xacro)
@@ -9,17 +9,7 @@
       <visual>
         <geometry>
-          <cylinder length="0.150" radius="0.029"/>
-        </geometry>
-        <origin rpy="${M_PI/2} 0 0"/>
-        <material name="polycarb">
-          <color rgba="1 1 1 0.3"/>
-        </material>
-      </visual>
-    </link>
-    <link name="${name}_pcb">
-      <visual>
-        <geometry>
           <box size="0.002 0.070 .016"/>
         </geometry>
+        <origin xyz="0.001 0 0"/>
         <material name="gray">
           <color rgba="0.1 0.1 0.1 1"/>
@@ -53,11 +43,6 @@
     <link name="${name}_right_optical_frame">
     </link>
-    <joint name="${name}_to_${name}_pcb" type="fixed">
+    <joint name="${name}_to_${name}_left_frame" type="fixed">
       <parent link="${name}"/>
-      <child link="${name}_pcb"/>
-      <origin xyz="-0.010 0 0"/>
-    </joint>
-    <joint name="${name}_pcb_to_${name}_left_frame" type="fixed">
-      <parent link="${name}_pcb"/>
       <child link="${name}_left_frame"/>
       <origin xyz="${BOARD_THICKNESS/2 + LENS_LENGTH} ${INTEROCULAR/2} 0"/>
@@ -68,6 +53,6 @@
       <origin xyz="0 0 0" rpy="${-M_PI/2} 0 ${-M_PI/2}"/>
     </joint>
-    <joint name="${name}_pcb_to_${name}_right_frame" type="fixed">
-      <parent link="${name}_pcb"/>
+    <joint name="${name}_to_${name}_right_frame" type="fixed">
+      <parent link="${name}"/>
       <child link="${name}_right_frame"/>
       <origin xyz="${BOARD_THICKNESS/2 + LENS_LENGTH} ${-INTEROCULAR/2} 0"/>
